File: I2C-Encoder-Keys/I2C-Encoder-Keys.kicad_sch (KiCad schematic)
At the start: 45 parts, among them J1 JST-S6B-PH-SM4, J2 JST-S6B-PH-SM4, J3 PH 1x6-2.54mm, SW0 SW_SPST, SW1 SW_SPST, SW2 SW_SPST, SW3 SW_SPST, U1 MCP23008-xSO

Commit message: Added encoder knob
Parts:
- C1: LCSC Part # (none) -> C49678
- C2, C3, C4, C5, C6, C7, C8: LCSC Part # (none) -> C1710
- C9: LCSC Part # (none) -> C28323
- H1, H2, H3, H4, JP1, JP2, JP3, JP4, JP5, JP6: now left out of the parts list
- J1, J2: LCSC Part # (none) -> C265405
- R1, R10, R11, R12, R13, R14, R15, R16, R17, R2, R3, R4, R5, R6, R7, R8, R9: LCSC Part # (none) -> C17414
- U1: LCSC Part # (none) -> C92253
Changed lines of the file:
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@@
   )
   (symbol (lib_id "Mechanical:MountingHole") (at 162.56 186.69 0) (unit 1)
-    (in_bom yes) (on_board yes) (fields_autoplaced)
+    (in_bom no) (on_board yes) (fields_autoplaced)
     (property "Reference" "H3" (id 0) (at 165.1 185.4199 0)
       (effects (font (size 1.27 1.27)) (justify left))
@@
       (effects (font (size 1.27 1.27)) hide)
     )
+    (property "LCSC Part #" "C1710" (id 4) (at 193.04 56.515 0)
+      (effects (font (size 1.27 1.27)) hide)
+    )
     (pin "1")
     (pin "2")
@@
       (effects (font (size 1.27 1.27)) hide)
     )
+    (property "LCSC Part #" "C1710" (id 4) (at 139.7 82.55 0)
+      (effects (font (size 1.27 1.27)) hide)
+    )
     (pin "1")
     (pin "2")
   )
   (symbol (lib_id "Jumper:Jumper_3_Bridged12") (at 86.36 89.535 180) (unit 1)
-    (in_bom yes) (on_board yes) (fields_autoplaced)
+    (in_bom no) (on_board yes) (fields_autoplaced)
     (property "Reference" "JP5" (id 0) (at 86.36 92.71 0))
     (property "Value" "A0" (id 1) (at 86.36 95.25 0))
@@
   )
   (symbol (lib_id "Jumper:Jumper_3_Bridged12") (at 59.69 71.12 180) (unit 1)
-    (in_bom yes) (on_board yes) (fields_autoplaced)
+    (in_bom no) (on_board yes) (fields_autoplaced)
     (property "Reference" "JP1" (id 0) (at 59.69 74.93 0))
     (property "Value" "A2" (id 1) (at 59.69 77.47 0))
@@
       (effects (font (size 1.27 1.27)) hide)
     )
+    (property "LCSC Part #" "C17414" (id 4) (at 64.77 35.56 0)
+      (effects (font (size 1.27 1.27)) hide)
+    )
     (pin "1")
     (pin "2")
@@
       (effects (font (size 1.27 1.27)) hide)
     )
+    (property "LCSC Part #" "C49678" (id 4) (at 128.905 33.655 0)
+      (effects (font (size 1.27 1.27)) hide)
+    )
     (pin "1")
     (pin "2")
   )
   (symbol (lib_id "Jumper:SolderJumper_2_Bridged") (at 89.535 43.815 90) (unit 1)
-    (in_bom yes) (on_board yes) (fields_autoplaced)
+    (in_bom no) (on_board yes) (fields_autoplaced)
     (property "Reference" "JP6" (id 0) (at 91.44 42.5449 90)
       (effects (font (size 1.27 1.27)) (justify right))
@@
   )
   (symbol (lib_id "Mechanical:MountingHole") (at 162.56 192.405 0) (unit 1)
-    (in_bom yes) (on_board yes) (fields_autoplaced)
+    (in_bom no) (on_board yes) (fields_autoplaced)
     (property "Reference" "H4" (id 0) (at 165.1 191.1349 0)
       (effects (font (size 1.27 1.27)) (justify left))
@@
     )
     (property "Datasheet" "http://ww1.microchip.com/downloads/en/DeviceDoc/MCP23008-MCP23S08-Data-Sheet-20001919F.pdf" (id 3) (at 141.605 90.805 0)
+      (effects (font (size 1.27 1.27)) hide)
+    )
+    (property "LCSC Part #" "C92253" (id 4) (at 108.585 60.325 0)
       (effects (font (size 1.27 1.27)) hide)
     )
@@
   )
   (symbol (lib_id "Jumper:SolderJumper_2_Bridged") (at 77.47 43.815 90) (unit 1)
-    (in_bom yes) (on_board yes) (fields_autoplaced)
+    (in_bom no) (on_board yes) (fields_autoplaced)
     (property "Reference" "JP4" (id 0) (at 80.01 42.5449 90)
       (effects (font (size 1.27 1.27)) (justify right))
@@
     )
     (property "Datasheet" "~" (id 3) (at 146.05 56.515 0)
+      (effects (font (size 1.27 1.27)) hide)
+    )
+    (property "LCSC Part #" "C1710" (id 4) (at 146.05 56.515 0)
       (effects (font (size 1.27 1.27)) hide)
     )
@@
     )
     (property "Datasheet" "~" (id 3) (at 154.94 50.8 0)
+      (effects (font (size 1.27 1.27)) hide)
+    )
+    (property "LCSC Part #" "C17414" (id 4) (at 154.94 50.8 0)
       (effects (font (size 1.27 1.27)) hide)
     )
@@
       (effects (font (size 1.27 1.27)) hide)
     )
+    (property "LCSC Part #" "C265405" (id 4) (at 26.67 78.105 0)
+      (effects (font (size 1.27 1.27)) hide)
+    )
     (pin "1")
     (pin "2")
@@
       (effects (font (size 1.27 1.27)) hide)
     )
+    (property "LCSC Part #" "C17414" (id 4) (at 89.535 35.56 0)
+      (effects (font (size 1.27 1.27)) hide)
+    )
     (pin "1")
     (pin "2")
@@
     )
     (property "Datasheet" "~" (id 3) (at 163.195 100.33 0)
+      (effects (font (size 1.27 1.27)) hide)
+    )
+    (property "LCSC Part #" "C17414" (id 4) (at 163.195 100.33 0)
       (effects (font (size 1.27 1.27)) hide)
     )
@@
       (effects (font (size 1.27 1.27)) hide)
     )
+    (property "LCSC Part #" "C17414" (id 4) (at 179.705 43.815 0)
+      (effects (font (size 1.27 1.27)) hide)
+    )
     (pin "1")
     (pin "2")
@@
       (effects (font (size 1.27 1.27)) hide)
     )
+    (property "LCSC Part #" "C17414" (id 4) (at 159.385 145.415 0)
+      (effects (font (size 1.27 1.27)) hide)
+    )
     (pin "1")
     (pin "2")
@@
   )
   (symbol (lib_id "Mechanical:MountingHole") (at 162.56 180.975 0) (unit 1)
-    (in_bom yes) (on_board yes) (fields_autoplaced)
+    (in_bom no) (on_board yes) (fields_autoplaced)
     (property "Reference" "H2" (id 0) (at 165.1 179.7049 0)
       (effects (font (size 1.27 1.27)) (justify left))
@@
     )
     (property "Datasheet" "~" (id 3) (at 159.385 43.815 0)
+      (effects (font (size 1.27 1.27)) hide)
+    )
+    (property "LCSC Part #" "C17414" (id 4) (at 159.385 43.815 0)
       (effects (font (size 1.27 1.27)) hide)
     )
@@
       (effects (font (size 1.27 1.27)) hide)
     )
+    (property "LCSC Part #" "C17414" (id 4) (at 213.995 100.33 0)
+      (effects (font (size 1.27 1.27)) hide)
+    )
     (pin "1")
     (pin "2")
@@
       (effects (font (size 1.27 1.27)) hide)
     )
+    (property "LCSC Part #" "C17414" (id 4) (at 77.47 35.56 0)
+      (effects (font (size 1.27 1.27)) hide)
+    )
     (pin "1")
     (pin "2")
@@
     )
     (property "Datasheet" "~" (id 3) (at 153.035 69.85 0)
+      (effects (font (size 1.27 1.27)) hide)
+    )
+    (property "LCSC Part #" "C17414" (id 4) (at 153.035 69.85 0)
       (effects (font (size 1.27 1.27)) hide)
     )
@@
       (effects (font (size 1.27 1.27)) hide)
     )
+    (property "LCSC Part #" "C17414" (id 4) (at 148.59 76.835 0)
+      (effects (font (size 1.27 1.27)) hide)
+    )
     (pin "1")
     (pin "2")
   )
   (symbol (lib_id "Jumper:Jumper_3_Bridged12") (at 73.025 80.01 180) (unit 1)
-    (in_bom yes) (on_board yes) (fields_autoplaced)
+    (in_bom no) (on_board yes) (fields_autoplaced)
     (property "Reference" "JP3" (id 0) (at 73.025 83.82 0))
     (property "Value" "A1" (id 1) (at 73.025 86.36 0))
@@
       (effects (font (size 1.27 1.27)) hide)
     )
+    (property "LCSC Part #" "C17414" (id 4) (at 214.63 136.525 0)
+      (effects (font (size 1.27 1.27)) hide)
+    )
     (pin "1")
     (pin "2")
@@
       (effects (font (size 1.27 1.27)) hide)
     )
+    (property "LCSC Part #" "C17414" (id 4) (at 210.185 143.51 0)
+      (effects (font (size 1.27 1.27)) hide)
+    )
     (pin "1")
     (pin "2")
@@
       (effects (font (size 1.27 1.27)) hide)
     )
+    (property "LCSC Part #" "C1710" (id 4) (at 200.66 113.03 0)
+      (effects (font (size 1.27 1.27)) hide)
+    )
     (pin "1")
     (pin "2")
@@
     )
     (property "Datasheet" "~" (id 3) (at 163.83 138.43 0)
+      (effects (font (size 1.27 1.27)) hide)
+    )
+    (property "LCSC Part #" "C17414" (id 4) (at 163.83 138.43 0)
       (effects (font (size 1.27 1.27)) hide)
     )
@@
     )
     (property "Datasheet" "~" (id 3) (at 55.245 33.655 0)
+      (effects (font (size 1.27 1.27)) hide)
+    )
+    (property "LCSC Part #" "C28323" (id 4) (at 55.245 33.655 0)
       (effects (font (size 1.27 1.27)) hide)
     )
@@
       (effects (font (size 1.27 1.27)) hide)
     )
+    (property "LCSC Part #" "C265405" (id 4) (at 26.67 55.245 0)
+      (effects (font (size 1.27 1.27)) hide)
+    )
     (pin "1")
     (pin "2")
@@
       (effects (font (size 1.27 1.27)) hide)
     )
+    (property "LCSC Part #" "C17414" (id 4) (at 209.55 107.315 0)
+      (effects (font (size 1.27 1.27)) hide)
+    )
     (pin "1")
     (pin "2")
@@
       (effects (font (size 1.27 1.27)) hide)
     )
+    (property "LCSC Part #" "C17414" (id 4) (at 158.75 107.315 0)
+      (effects (font (size 1.27 1.27)) hide)
+    )
     (pin "1")
     (pin "2")
@@
       (effects (font (size 1.27 1.27)) hide)
     )
+    (property "LCSC Part #" "C17414" (id 4) (at 184.15 50.8 0)
+      (effects (font (size 1.27 1.27)) hide)
+    )
     (pin "1")
     (pin "2")
   )
   (symbol (lib_id "Mechanical:MountingHole") (at 162.56 175.26 0) (unit 1)
-    (in_bom yes) (on_board yes) (fields_autoplaced)
+    (in_bom no) (on_board yes) (fields_autoplaced)
     (property "Reference" "H1" (id 0) (at 165.1 173.9899 0)
       (effects (font (size 1.27 1.27)) (justify left))
@@
       (effects (font (size 1.27 1.27)) hide)
     )
+    (property "LCSC Part #" "C1710" (id 4) (at 201.295 149.225 0)
+      (effects (font (size 1.27 1.27)) hide)
+    )
     (pin "1")
     (pin "2")
   )
   (symbol (lib_id "Jumper:SolderJumper_2_Bridged") (at 64.77 43.815 90) (unit 1)
-    (in_bom yes) (on_board yes) (fields_autoplaced)
+    (in_bom no) (on_board yes) (fields_autoplaced)
     (property "Reference" "JP2" (id 0) (at 67.31 42.5449 90)
       (effects (font (size 1.27 1.27)) (justify right))
@@
       (effects (font (size 1.27 1.27)) hide)
     )
+    (property "LCSC Part #" "C1710" (id 4) (at 149.86 113.03 0)
+      (effects (font (size 1.27 1.27)) hide)
+    )
     (pin "1")
     (pin "2")
@@
       (effects (font (size 1.27 1.27)) hide)
     )
+    (property "LCSC Part #" "C1710" (id 4) (at 150.495 151.13 0)
+      (effects (font (size 1.27 1.27)) hide)
+    )
